File: source/usbpowerios.kicad_sch (KiCad schematic)
At the start: 46 parts, among them J1 TYPE-C-31-M-12, J2 GSB343133HR, J3 PZ254V-12-14P, SW1 Tactile Switch, SW2 Tactile Switch, SW3 Tactile Switch, U1 USBLC6-2SC6Y, U2 SC1556, U3 USBLC6-2SC6Y, U4 USBLC6-2SC6Y, U5 AP22653W6-7

Commit message: schematics r1 done, awaiting verification
Parts:
- removed J2: GSB343133HR, nielo:AMPHENOL_GSB343133HR, symbol nielo:GSB343133HR
- removed U4: USBLC6-2SC6Y, nielo:SOT23-6L_STM, symbol nielo:USBLC6-2SC6Y
- added B5: PESD5V5C1BLYL, nielo:PESD5V5C1BLYL, symbol nielo:PESD5V5C1BLYL
- added BT1: BS-07-A1BJ001, nielo:BatteryHolder_MYOUNG_BS-07-A1BJ001_CR2032, symbol nielo:BS-07-A1BJ001
- added C18: 10u 50V, nielo:CAPC2012X11L, symbol nielo:C0805
- added HS1: SC1752, symbol nielo:SC1752
- added J2: TYPE-C-31-M-12, nielo:HRO_TYPE-C-31-M-12, symbol nielo:TYPE-C-31-M-12
- added R24, R25: 5k1, nielo:RESC1005X04L, symbol nielo:R0402
- C1, C13, C15, C2, C5, C8: DigiKey No (none) -> 478-KGM05CR71H104JHTR-ND; LCSC No (none) -> C2169023; MPN (none) -> 04025C104JAT2A; Mouser No (none) -> 581-04025C104JAT2A
- C10, C9: DigiKey No (none) -> 13-CC0603KRX5R8BB106TR-ND; LCSC No (none) -> C7500379; MPN (none) -> CC0603KRX5R8BB106; Mouser No (none) -> 603-CC0603KRX5R8BB10
- C11: DigiKey No (none) -> 738-CML0603X7R104KT50VTR-ND; LCSC No (none) -> C2594245; MPN (none) -> CML0603X7R104KT50V; Mouser No (none) -> 708-CML0603X7R104K50
- C3, C4, C6, C7: value N.C. -> TBD; MPN (none) -> TBD
- D4: DigiKey No (none) -> 1080-16-213/GHC-YR1S1/3TTR-ND; Mouser No (none) -> 638-16213GHCYR1S13T
- R1, R2: DigiKey No (none) -> 541-3156-2-ND; LCSC No (none) -> C2088796; MPN (none) -> TNPW04025K10BEED; Mouser No (none) -> 71-TNPW04025K10BEED
- R10, R9: LCSC No (none) -> C2076615; MPN (none) -> CRCW04021K65FKEE; Mouser No (none) -> 71-CRCW04021K65FKEE
- R22, R23, R6: DigiKey No (none) -> 749-MCS0402MD1002BE500TR-ND; LCSC No (none) -> C2073498; MPN (none) -> MCS0402MD1002BE500; Mouser No (none) -> 594-MCS0402MD1002BE5
- R3, R4, R7, R8: DigiKey No (none) -> CR0402-JW-220GLFTR-ND; LCSC No (none) -> C2076445; MPN (none) -> CR0402-JW-220GLF; Mouser No (none) -> 652-CR0402-JW-220GLF
- R5: DigiKey No (none) -> 749-MCS04020C1502FE500TR-ND; LCSC No (none) -> C2074222; MPN (none) -> MCS04020C1502FE500; Mouser No (none) -> 594-MCS04020C1502FE5
- TP1: now left out of the parts list
Connections:
- net GND: now also B5.1 (K1), BT1.2 (-), C18.2, J2.A1_B12 (GND), J2.B1_A12 (GND), J2.S1, J2.S2, J2.S3, J2.S4, R24.2, R25.2
- net VBUS_SS: now also J2.A4_B9 (VBUS), J2.B4_A9 (VBUS)
- net _usb_ss-n: now also J2.A7 (DN1), J2.B7 (DN2)
- net _usb_ss-p: now also J2.A6 (DP1), J2.B6 (DP2)
- net +VBAT: now reaches U2.76 (VBAT)
- net +VBAT: now also B5.2 (K2), BT1.1 (+), C18.1
- net cc1 renamed cc1_hs
- net cc2 renamed cc2_hs
- net sync_out: no longer names the net of J3.6
- net usb_ss_rx-n: no longer names the net of U2.157 (USB3-1-RX_N)
- net usb_ss_rx-n: no longer U3.3 (I/O2)
- net usb_ss_rx-p: no longer names the net of U2.159 (USB3-1-RX_P)
- net usb_ss_rx-p: no longer U3.6 (I/O1)
- net usb_ss_tx-n: no longer names the net of U2.169 (USB3-1-TX_N)
- net usb_ss_tx-p: no longer names the net of U2.171 (USB3-1-TX_P)
- new net cc1_ss: J2.A5 (CC1), R24.1
- new net cc2_ss: J2.B5 (CC2), R25.1
- no-connect marks 98 -> 127
Other:
- moved on the sheet: B2, C13, C15, C5, C8, D2, R1, R2, R22, R23, R6, SW1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
