File: source/usbpowerios.kicad_sch (KiCad schematic)
At the start: 51 parts, among them J1 TYPE-C-31-M-12, J2 TYPE-C-31-M-12, J3 PZ254V-12-14P, SW1 Tactile Switch, SW2 Tactile Switch, SW3 Tactile Switch, U1 USBLC6-2SC6Y, U2 SC1556, U3 USBLC6-2SC6Y, U5 AP22653W6-7

Commit message: layout done, awaiting verification
Parts:
- added H1, H2, H3, H4: MountingHole_Pad, nielo:MountingHole_3.2mm_M3_Pad_Via, symbol nielo:MountingHole_Pad
Connections:
- net GND: now also H1.1, H2.1, H3.1, H4.1
- net _usb_hs-n renamed _usb_hs-
- net _usb_hs-p renamed _usb_hs+
- net _usb_ss-n renamed _usb_ss-
- net _usb_ss-p renamed _usb_ss+
- net usb_hs-n renamed usb_hs-
- net usb_hs-p renamed usb_hs+
- net usb_ss-n renamed usb_ss-
- net usb_ss-p renamed usb_ss+

Commit message: mounting holes flash
Parts:
- H1, H2, H3, H4: footprint nielo:MountingHole_3.2mm_M3_Pad_Via -> nielo:MountingHole_2.2mm_M2_Pad_Via
Connections:
- net VBUS_HS: no longer U3.5 (VBUS)
- net VBUS_SS: now also U3.5 (VBUS)
Changed lines of the file:
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@@
 			)
 		)
-		(property "Footprint" "nielo:MountingHole_3.2mm_M3_Pad_Via"
+		(property "Footprint" "nielo:MountingHole_2.2mm_M2_Pad_Via"
 			(at 430.53 322.58 0)
 			(hide yes)
@@
 			)
 		)
-		(property "Footprint" "nielo:MountingHole_3.2mm_M3_Pad_Via"
+		(property "Footprint" "nielo:MountingHole_2.2mm_M2_Pad_Via"
 			(at 467.36 322.58 0)
 			(hide yes)
@@
 			)
 		)
-		(property "Footprint" "nielo:MountingHole_3.2mm_M3_Pad_Via"
+		(property "Footprint" "nielo:MountingHole_2.2mm_M2_Pad_Via"
 			(at 542.29 322.58 0)
 			(hide yes)
@@
 			)
 		)
-		(property "Value" "VBUS_HS"
-			(at 62.23 273.05 0)
+		(property "Value" "VBUS_SS"
+			(at 64.77 276.8599 0)
 			(show_name no)
 			(do_not_autoplace no)
@@
 					(size 1.27 1.27)
 				)
+				(justify left)
 			)
 		)
@@
 			)
 		)
-		(property "Footprint" "nielo:MountingHole_3.2mm_M3_Pad_Via"
+		(property "Footprint" "nielo:MountingHole_2.2mm_M2_Pad_Via"
 			(at 501.65 322.58 0)
 			(hide yes)

Commit message: manufactering files & step files added
Parts:
- removed D1: SS54FSH, nielo:SODFL4725X110N, symbol nielo:SS54F
- added J4, J9: 10164227-1001A1RLF, symbol nielo:10164227-1001A1RLF
- C3, C4, C6, C7: now left out of the parts list
- R24, R25: value 5k1 -> 10k; DigiKey No 541-3156-2-ND -> 749-MCS0402MD1002BE500TR-ND; LCSC No C2088796 -> C2073498; MPN TNPW04025K10BEED -> MCS0402MD1002BE500; Mouser No 71-TNPW04025K10BEED -> 594-MCS0402MD1002BE5
Connections:
- net +3V3: now also R24.2, R25.2
- net GND: no longer R24.2, R25.2
- net VBUS_HS: now also C1.2, FB1.1
- no-connect marks 127 -> 327

Commit message: usbss pull-up resistors 10k-->12k
Parts:
- R24, R25: value 10k -> 12k; DigiKey No 749-MCS0402MD1002BE500TR-ND -> CR0402-FX-1202GLFTR-ND; LCSC No C2073498 -> C2085429; MPN MCS0402MD1002BE500 -> CR0402-FX-1202GLF; Mouser No 594-MCS0402MD1002BE5 -> 652-CR0402FX-1202GLF
Other:
- moved on the sheet: HS1
Changed lines of the file:
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@@
 	(symbol
 		(lib_id "nielo:SC1752")
-		(at 556.26 184.15 0)
+		(at 556.26 109.22 0)
 		(unit 1)
 		(body_style 1)
@@
 		(dnp no)
 		(property "Reference" "HS1"
-			(at 553.72 177.038 0)
+			(at 553.72 102.108 0)
 			(show_name no)
 			(do_not_autoplace no)
@@
 				(font
 					(size 1.778 1.778)
-					(color 255 77 92 1)
+					(color 0 0 0 1)
 				)
 				(justify left)
@@
 		)
 		(property "Value" "SC1752"
-			(at 551.688 187.452 0)
+			(at 551.688 112.522 0)
 			(show_name no)
 			(do_not_autoplace no)
@@
 				(font
 					(size 1.778 1.778)
-					(color 255 77 92 1)
+					(color 0 0 0 1)
 				)
 				(justify left)
@@
 		)
 		(property "Footprint" ""
-			(at 556.5648 184.15 0)
+			(at 556.5648 109.22 0)
 			(hide yes)
 			(show_name no)
@@
 		)
 		(property "Datasheet" ""
-			(at 556.5648 184.15 0)
+			(at 556.5648 109.22 0)
 			(hide yes)
 			(show_name no)
@@
 		)
 		(property "Description" "Heat Sink Raspberry Pi 5 Aluminum Top Mount"
-			(at 556.26 184.15 0)
+			(at 556.26 109.22 0)
 			(hide yes)
 			(show_name no)
@@
 		)
 		(property "MPN" "SC1752"
-			(at 556.26 184.15 0)
+			(at 556.26 109.22 0)
 			(hide yes)
 			(show_name no)
@@
 		)
 		(property "Mouser No" "358-SC1752"
-			(at 556.26 184.15 0)
+			(at 556.26 109.22 0)
 			(hide yes)
 			(show_name no)
@@
 		)
 		(property "DigiKey No" "2648-SC1752-ND"
-			(at 556.26 184.15 0)
+			(at 556.26 109.22 0)
 			(hide yes)
 			(show_name no)
@@
 		)
 		(property "LCSC No" ""
-			(at 556.26 184.15 0)
+			(at 556.26 109.22 0)
 			(hide yes)
 			(show_name no)
@@
 			)
 		)
-		(property "Value" "10k"
+		(property "Value" "12k"
 			(at 98.044 245.11 0)
 			(show_name no)
@@
 			)
 		)
-		(property "Description" "10k Resistor Ceramic 0402"
+		(property "Description" "12k Resistor Ceramic 0402"
 			(at 92.71 242.57 0)
 			(hide yes)
@@
 			)
 		)
-		(property "LCSC No" "C2073498"
+		(property "LCSC No" "C2085429"
 			(at 87.122 251.206 0)
 			(hide yes)
@@
 			)
 		)
-		(property "DigiKey No" "749-MCS0402MD1002BE500TR-ND"
+		(property "DigiKey No" "CR0402-FX-1202GLFTR-ND"
 			(at 87.122 248.666 0)
 			(hide yes)
@@
 			)
 		)
-		(property "Mouser No" "594-MCS0402MD1002BE5"
+		(property "Mouser No" "652-CR0402FX-1202GLF"
 			(at 87.122 248.666 0)
 			(hide yes)
@@
 			)
 		)
-		(property "MPN" "MCS0402MD1002BE500"
+		(property "MPN" "CR0402-FX-1202GLF"
 			(at 87.122 248.666 0)
 			(hide yes)
@@
 			)
 		)
-		(property "Value" "10k"
+		(property "Value" "12k"
 			(at 97.79 237.236 0)
 			(show_name no)
@@
 			)
 		)
-		(property "Description" "10k Resistor Ceramic 0402"
+		(property "Description" "12k Resistor Ceramic 0402"
 			(at 92.71 240.03 0)
 			(hide yes)
@@
 			)
 		)
-		(property "LCSC No" "C2073498"
+		(property "LCSC No" "C2085429"
 			(at 87.122 248.666 0)
 			(hide yes)
@@
 			)
 		)
-		(property "DigiKey No" "749-MCS0402MD1002BE500TR-ND"
+		(property "DigiKey No" "CR0402-FX-1202GLFTR-ND"
 			(at 87.122 246.126 0)
 			(hide yes)
@@
 			)
 		)
-		(property "Mouser No" "594-MCS0402MD1002BE5"
+		(property "Mouser No" "652-CR0402FX-1202GLF"
 			(at 87.122 246.126 0)
 			(hide yes)
@@
 			)
 		)
-		(property "MPN" "MCS0402MD1002BE500"
+		(property "MPN" "CR0402-FX-1202GLF"
 			(at 87.122 246.126 0)
 			(hide yes)
