File: source/nielo.kicad_pcb (KiCad board)
At the start: 6 copper layers, 98 x 98 mm, 102 parts, among them J1 TYPE-C-31-M-12, J2 TYPE-C-31-M-12, J3 PZ254V-12-14P, J5 SM04B-SRSS-TB, J6 SM04B-SRSS-TB, J7 SM04B-SRSS-TB, J8 SM04B-SRSS-TB, Q1 AO3401A, Q2 2N7002, Q3 2N7002, Q4 AO3401A, SW1 Tactile Switch, SW2 Tactile Switch, SW3 Tactile Switch, U1 USBLC6-2SC6Y, U2 SC1556, U3 USBLC6-2SC6Y, U5 AP22653W6-7, U6 SN74AHCT1G125DBVR, U7 SN74AHCT1G125DBVR

Commit message: usb pair routed
Parts:
- moved B2 0.44 mm to (205.8, 73.6)
Routing:
- net /usbpowerios/usb_hs+: track 3.69 -> 63.8 mm, vias 1 -> 2
- net /usbpowerios/usb_hs-: track 3.56 -> 63.2 mm, vias 1 -> 2
- net /usbpowerios/usb_ss-: track 0.00 -> 27.8 mm, vias 0 -> 2
- net /usbpowerios/usb_ss+: track 0.00 -> 27.6 mm, vias 0 -> 2
- net /usbpowerios/_usb_ss-: track 0.00 -> 7.11 mm
- net /usbpowerios/_usb_ss+: track 0.00 -> 6.55 mm
- net VBUS_SS: track 0.00 -> 6.33 mm
- net GND: track 6.94 -> 9.67 mm

Commit message: mounting holes flash
Parts:
- H1, H3, H4: footprint nielo:MountingHole_3.2mm_M3_Pad_Via -> nielo:MountingHole_2.2mm_M2_Pad_Via
- H2: footprint nielo:MountingHole_3.2mm_M3_Pad_Via -> nielo:MountingHole_2.2mm_M2_Pad_Via; moved to B.Cu
- moved H2 19.0 mm to (140.7, 57.3), turned to 180 degrees
- moved H1 16.7 mm to (199.2, 78.6)
- moved R25 11.0 mm to (210.3, 73.1)
- moved R24 10.9 mm to (210.3, 84.2), turned to 180 degrees
- moved H3 6.24 mm to (140.7, 100.0)
- moved R10 4.83 mm to (141.9, 53.7)
- moved D4 4.69 mm to (141.9, 52.4)
- moved C6 1.90 mm to (203.2, 80.5), turned to 0 degrees
- moved C7 1.89 mm to (203.2, 76.8), turned to 180 degrees
- moved J6 0.20 mm to (132.4, 46.5)
Connections:
- C17 pad 2: +3V3_i2c -> +3V3_uart
- D6 pad C: +3V3_i2c -> +3V3_uart
- J7 pad 1: +3V3_i2c -> +3V3_uart
- TP11 pad 1: i2c_dbg_scl -> i2c_dbg_sda
- U3 pad 5: VBUS_HS -> VBUS_SS
Routing:
- net GND: track 9.67 -> 128.2 mm, vias 0 -> 96
- net vbus_en: track 0.00 -> 82.1 mm, vias 0 -> 3
- net /usbpowerios/pwr_but: track 0.00 -> 78.3 mm, vias 0 -> 5
- net /usbpowerios/usb_otg_id: track 0.00 -> 76.5 mm, vias 0 -> 1
- net /usbpowerios/eeprom_nwp: track 0.00 -> 75.0 mm, vias 0 -> 3
- net led_pwr_en: track 0.00 -> 72.2 mm, vias 0 -> 4
- net fan_tacho: track 0.00 -> 65.8 mm, vias 0 -> 2
- net /usbpowerios/btn_mute: track 0.00 -> 65.6 mm, vias 0 -> 2
- net led_clk_3v3: track 0.00 -> 64.8 mm, vias 0 -> 4
- net /usbpowerios/n_rpiboot: track 0.00 -> 60.8 mm, vias 0 -> 3
- net fan_pwm: track 0.00 -> 60.0 mm, vias 0 -> 2
- net uart_dbg_tx: track 0.00 -> 60.0 mm, vias 0 -> 2
- net uart_dbg_rx: track 0.00 -> 59.4 mm, vias 0 -> 2
- net /usbpowerios/pmic_en: track 0.00 -> 58.4 mm, vias 0 -> 1
- net led_dat_3v3: track 0.00 -> 55.6 mm, vias 0 -> 4
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- added copper zone on In2.Cu, net +3V3
- added copper zone on In1.Cu, net GND
- added copper zone on In3.Cu, net GND
- added copper zone on In4.Cu, net GND
- added copper zone on F.Cu, net VUSB_HS
- added copper zone on B.Cu, net VUSB_SS
