File: source/peripherals.kicad_sch (KiCad schematic)
At the start: 41 parts, among them J5 SM04B-SRSS-TB, J6 SM04B-SRSS-TB, J7 SM04B-SRSS-TB, J8 SM04B-SRSS-TB, Q1 AO3401A, Q2 2N7002, Q3 2N7002, Q4 AO3401A, U6 SN74AHCT1G125DBVR, U7 SN74AHCT1G125DBVR

Commit message: schematics r1 done, awaiting verification
Parts:
- removed TP3, TP4, TP8, TP9: TP_SMD_D1.5mm, nielo:TP_SMD_D1.5mm, symbol nielo:TP_SMD_Ø1.5MM
- C12, C14, C16, C17: DigiKey No (none) -> 478-KGM05CR71H104JHTR-ND; LCSC No (none) -> C2169023; MPN (none) -> 04025C104JAT2A; Mouser No (none) -> 581-04025C104JAT2A
- R11, R12, R15, R16, R17, R18: DigiKey No (none) -> CR0402-JW-104GLFTR-ND; LCSC No (none) -> C203104; MPN (none) -> CR0402-JW-104GLF; Mouser No (none) -> 652-CR0402JW-104GLF
- R13, R14: DigiKey No (none) -> 749-MCS0402MC3309FE000TR-ND; LCSC No (none) -> C2074234; MPN (none) -> MCS0402MC3309FE000; Mouser No (none) -> 594-MCS0402MC3309FE0
- R19: DigiKey No (none) -> 749-MCS0402MD1002BE500TR-ND; LCSC No (none) -> C2073498; MPN (none) -> MCS0402MD1002BE500; Mouser No (none) -> 594-MCS0402MD1002BE5
- R20, R21: DigiKey No (none) -> 541-RCA04024K70FKEDSRTR-ND; LCSC No (none) -> C1858949; MPN (none) -> RCA04024K70FKED; Mouser No (none) -> 594-RCA04024K70FKED
Connections:
- net GND: now also J5.4; no longer J5.3
- net fan_tacho: now also J5.3; no longer J5.4
- net i2c_dbg_sda: no longer J6.3, R20.1, TP10.1, TP11.1
- new net i2c_dbg_scl: J6.3, R20.1, TP10.1, TP11.1
Other:
- note added: "DEBUG INTERFACEs"
- note removed: "DEBUG INTERFACE"

Commit message: layout done, awaiting verification
Connections:
- net uart_dbg_rx: no longer TP13.1
- net uart_dbg_tx: now also TP13.1
Changed lines of the file:
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@@
+	)
+	(junction
+		(at 92.71 294.64)
+		(diameter 0)
+		(color 0 0 0 0)
 	)
 	(junction
@@
 	(junction
 		(at 254 298.45)
-		(diameter 0)
-		(color 0 0 0 0)
-	)
-	(junction
-		(at 92.71 297.18)
 		(diameter 0)
 		(color 0 0 0 0)
@@
 	(wire
 		(pts
-			(xy 71.12 294.64) (xy 106.68 294.64)
+			(xy 71.12 294.64) (xy 92.71 294.64)
 		)
 		(stroke
@@
 	(wire
 		(pts
-			(xy 92.71 314.96) (xy 92.71 297.18)
-		)
-		(stroke
-			(width 0)
-			(type default)
-		)
-	)
-	(wire
-		(pts
 			(xy 353.06 158.75) (xy 369.57 158.75)
 		)
@@
 	(wire
 		(pts
+			(xy 92.71 294.64) (xy 106.68 294.64)
+		)
+		(stroke
+			(width 0)
+			(type default)
+		)
+	)
+	(wire
+		(pts
 			(xy 284.48 295.91) (xy 287.02 295.91)
 		)
@@
 	(wire
 		(pts
+			(xy 92.71 294.64) (xy 92.71 314.96)
+		)
+		(stroke
+			(width 0)
+			(type default)
+		)
+	)
+	(wire
+		(pts
 			(xy 243.84 271.78) (xy 243.84 275.59)
 		)
@@
 		)
 	)
-	(wire
-		(pts
-			(xy 92.71 297.18) (xy 106.68 297.18)
-		)
-		(stroke
-			(width 0)
-			(type default)
-		)
-	)
 	(bus
 		(pts
@@
 	(wire
 		(pts
-			(xy 83.82 297.18) (xy 92.71 297.18)
-		)
-		(stroke
+			(xy 83.82 297.18) (xy 106.68 297.18)
+		)
+		(stroke

Commit message: mounting holes flash
Connections:
- net +3V3_i2c: no longer C17.2, D6.C (K), J7.1
- net i2c_dbg_scl: no longer TP11.1
- net i2c_dbg_sda: now also TP11.1
- new net +3V3_uart: C17.2, D6.C (K), J7.1
Changed lines of the file:
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@@
-	)
-	(junction
-		(at 254 300.99)
-		(diameter 0)
-		(color 0 0 0 0)
 	)
 	(junction
@@
 	(wire
 		(pts
+			(xy 254 298.45) (xy 254 322.58)
+		)
+		(stroke
+			(width 0)
+			(type default)
+		)
+	)
+	(wire
+		(pts
 			(xy 284.48 281.94) (xy 284.48 295.91)
 		)
@@
 	(wire
 		(pts
-			(xy 254 300.99) (xy 287.02 300.99)
+			(xy 243.84 300.99) (xy 287.02 300.99)
 		)
 		(stroke
@@
 	(wire
 		(pts
-			(xy 243.84 300.99) (xy 254 300.99)
-		)
-		(stroke
-			(width 0)
-			(type default)
-		)
-	)
-	(wire
-		(pts
 			(xy 185.42 74.93) (xy 201.93 74.93)
 		)
@@
 		(pts
 			(xy 353.06 223.52) (xy 369.57 223.52)
-		)
-		(stroke
-			(width 0)
-			(type default)
-		)
-	)
-	(wire
-		(pts
-			(xy 254 300.99) (xy 254 322.58)
 		)
 		(stroke
@@
 		(in_pos_files yes)
 		(dnp no)
-		(fields_autoplaced yes)
 		(property "Reference" "#PWR077"
 			(at 104.14 271.78 0)
@@
 			)
 		)
-		(property "Value" "+3V3_i2c"
-			(at 104.14 262.89 0)
+		(property "Value" "+3V3_uart"
+			(at 98.298 263.652 0)
 			(show_name no)
 			(do_not_autoplace no)
@@
 					(size 1.27 1.27)
 				)
-			)
-		)
+				(justify left)
+			)
+		)
